File: Project/ampersand.kicad_pcb (KiCad board)
At the start: 2 copper layers, 257.2 x 76.2 mm, 121 parts, among them J1 JST SH, SW1 DFU, U1 STM32F072CBT6, U2 XC6206PxxxMR-Regulator_Linear, U3 74HC4051, U4 OPA354, U5 74HC4051

Commit message: clean up
Parts:
- SW_EC40, SW_EC49: footprint cipulot_parts:ecs_pad_no_ring_stepped&normal_cut -> cipulot_parts:ecs_pad_no_ring_stepped&normal
- moved R3 3.24 mm to (131.6, 84.4)
- moved R4 2.80 mm to (131.6, 83.4)
- moved R1 2.80 mm to (131.6, 86.5)
- moved R2 2.68 mm to (131.6, 85.4)
- moved C1 1.28 mm to (92.5, 89.9)
- moved C10 1.28 mm to (37.9, 55.7)
- moved C11 1.28 mm to (50.3, 67.5)
- moved C12 1.28 mm to (96.8, 85.2)
- moved C13 1.28 mm to (91.5, 83.7)
- moved C14 1.28 mm to (197.9, 83.3)
- moved C2 1.28 mm to (102.7, 96.5)
- moved C3 1.28 mm to (95.3, 97.8)
- moved C4 1.28 mm to (93.9, 96.4)
- moved C5 1.28 mm to (102.2, 85.2)
- moved C6 1.28 mm to (102.8, 87.7)
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Connections:
- R2 pad 1: Net-(U1-PB4) -> Net-(U1-PB5)
- R2 pad 2: ROW0 -> ROW1
- R3 pad 1: Net-(U1-PB5) -> Net-(U1-PB4)
- R3 pad 2: ROW1 -> ROW0
Routing:
- net COL2: track 107.1 -> 92.7 mm, vias 4 -> 3
- net COL1: track 84.6 -> 71.8 mm, vias 5 -> 4
- net COL3: track 110.6 -> 98.1 mm
- net ROW3: track 408.5 -> 397.8 mm
- net COL11: track 170.6 -> 161.7 mm, vias 4 -> 1
- net ROW1: track 418.3 -> 424.8 mm
- net ROW0: track 433.4 -> 428.8 mm
- net ROW2: track 365.7 -> 362.0 mm
- net Net-(U1-PB3): track 41.3 -> 45.0 mm
- net Net-(U1-PB5): track 43.5 -> 47.2 mm
- net Net-(U1-PB6): track 44.6 -> 48.3 mm
- net Net-(U1-PB4): track 42.5 -> 46.1 mm
- net COL12: track 194.7 -> 191.6 mm, vias 5 -> 1
- net COL10: track 108.6 -> 105.5 mm, vias 5 -> 1
- net +3V3: track 278.0 -> 275.4 mm
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Other:
- outline, holes or cut-outs redrawn
- board text added: "1"
- board text added: "125"
- board text added: "150"
- board text added: "175"
- board text added: "225"
- board text added: "275"
- board text added: "3"
- board text added: "6 7 8 10"
- board text added: "ISO"
- board text added: "READD GND IN PADSS after trace clean!!!!!"
- board text added: "REDO COLUM ROUTING FOR CLEANER LOOK!!!!!!!"
- board text added: "og curves here!"
