File: Project/ampersand.kicad_pcb (KiCad board)
At the start: 2 copper layers, 257.2 x 76.2 mm, 125 parts, among them J1 JST SH, SW1 DFU, U1 STM32F072CBT6, U2 XC6206PxxxMR-Regulator_Linear, U3 74HC4051, U4 OPA354, U5 74HC4051

Commit message: v1 production files
Parts:
- added H28: MountingHole, cipulot_parts:HOLE_M2 (no arrow), F.Cu at (27.0, 81.8)
- added H29: MountingHole, cipulot_parts:HOLE_M2 (no arrow), F.Cu at (265.1, 81.8)
- H1, H10, H11, H12, H13, H14, H15, H16, H17, H18, H19, H2, H20, H21, H22, H23, H24, H25, H26, H27, H3, H4, H5, H6, H7, H8, H9: footprint cipulot_parts:HOLE_M2 -> cipulot_parts:HOLE_M2 (no arrow)
- moved H21 21.4 mm to (41.3, 53.2)
- moved H9 3.18 mm to (269.9, 34.1)
- moved H3 2.38 mm to (22.2, 72.2)
Routing:
- net ROW1: track 424.5 -> 414.5 mm
- net COL0: track 105.1 -> 106.3 mm

Commit message: update
error fixing
Routing:
- net ROW0: track 428.4 -> 427.7 mm, vias 14 -> 1
- net COL4: track 137.4 -> 136.9 mm, vias 7 -> 3
- net COL9: track 76.2 -> 75.8 mm, vias 5 -> 1
- net COL0: track 106.3 -> 106.0 mm, vias 6 -> 2
- net COL11: track 172.5 -> 172.1 mm, vias 4 -> 0
- net ROW2: track 362.0 -> 361.7 mm, vias 16 -> 3
- net COL12: track 196.8 -> 196.5 mm, vias 5 -> 0
- net COL10: track 107.1 -> 106.8 mm, vias 4 -> 0
- net COL2: track 101.1 -> 100.9 mm, vias 4 -> 0
- net COL7: track 76.1 -> 75.9 mm, vias 4 -> 0
- net COL8: track 56.6 -> 56.4 mm, vias 3 -> 0
- net COL6: track 101.1 -> 100.9 mm, vias 6 -> 2
- net COL5: track 141.6 -> 141.4 mm, vias 8 -> 5
- net COL3: track 95.4 -> 95.3 mm, vias 3 -> 0
- net COL1: track 71.7 -> 71.6 mm, vias 4 -> 0
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
Commit message: update production files
Routing:
- net ROW0: track 427.7 -> 428.2 mm
- net GND: vias 417 -> 421
Changed lines of the file:
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@@
 	)
 	(segment
-		(start 143.053744 62.650646)
-		(end 138.90625 62.650646)
+		(start 143.4625 63.5)
+		(end 143.4625 82.778064)
 		(width 0.2)
 		(layer "F.Cu")
@@
 	)
 	(segment
-		(start 141.80113 84.439434)
-		(end 143.4625 82.778064)
+		(start 138.224999 61.969395)
+		(end 138.90625 62.650646)
 		(width 0.2)
 		(layer "F.Cu")
@@
 	)
 	(segment
-		(start 143.4625 63.059402)
-		(end 143.053744 62.650646)
+		(start 140.176249 34.13125)
+		(end 138.224999 36.0825)
 		(width 0.2)
 		(layer "F.Cu")
@@
 	)
 	(segment
-		(start 133.399467 84.43338)
-		(end 133.405521 84.439434)
+		(start 133.405521 84.439434)
+		(end 133.399467 84.43338)
 		(width 0.2)
 		(layer "F.Cu")
@@
 	)
 	(segment
-		(start 132.894273 84.43338)
-		(end 133.399467 84.43338)
+		(start 138.90625 62.650646)
+		(end 142.613146 62.650646)
 		(width 0.2)
 		(layer "F.Cu")
@@
 	(segment
 		(start 138.224999 36.0825)
-		(end 140.176249 34.13125)
+		(end 138.224999 61.969395)
 		(width 0.2)
 		(layer "F.Cu")
@@
 	)
 	(segment
-		(start 138.90625 62.650646)
-		(end 138.224999 61.969395)
+		(start 143.4625 82.778064)
+		(end 141.80113 84.439434)
 		(width 0.2)
 		(layer "F.Cu")
@@
 	)
 	(segment
-		(start 138.224999 61.969395)
-		(end 138.224999 36.0825)
+		(start 142.613146 62.650646)
+		(end 143.4625 63.5)
 		(width 0.2)
 		(layer "F.Cu")
@@
 	)
 	(segment
-		(start 143.4625 82.778064)
-		(end 143.4625 63.059402)
+		(start 133.399467 84.43338)
+		(end 132.894273 84.43338)
 		(width 0.2)
 		(layer "F.Cu")
@@
 	)
 	(segment
-		(start 133.405521 84.439434)
-		(end 141.80113 84.439434)
+		(start 141.80113 84.439434)
+		(end 133.405521 84.439434)
 		(width 0.2)
 		(layer "F.Cu")
@@
 	(segment
 		(start 157.75 34.13125)
+		(end 159.3375 34.13125)
+		(width 0.5)
+		(layer "B.Cu")
+		(net 2)
+	)
+	(segment
+		(start 157.75 34.13125)
 		(end 156.95625 34.925)
 		(width 0.5)
@@
 	)
 	(segment
-		(start 158.54375 34.13125)
-		(end 157.75 34.13125)
-		(width 0.5)
-		(layer "B.Cu")
-		(net 2)
-	)
-	(segment
 		(start 238.692318 34.111068)
 		(end 239.50625 34.925)
@@
 	)
 	(via
+		(at 258.316035 82.98871)
+		(size 0.8)
+		(drill 0.4)
+		(layers "F.Cu" "B.Cu")
+		(free yes)
+		(net 3)
+	)
+	(via
 		(at 113.50625 96.04375)
 		(size 0.8)
@@
 	)
 	(via
+		(at 257.333943 81.706822)
+		(size 0.8)
+		(drill 0.4)
+		(layers "F.Cu" "B.Cu")
+		(free yes)
+		(net 3)
+	)
+	(via
 		(at 187.77414 41.124871)
 		(size 0.8)
@@
 	)
 	(via
+		(at 33.860851 82.59652)
+		(size 0.8)
+		(drill 0.4)
+		(layers "F.Cu" "B.Cu")
+		(free yes)
+		(net 3)
+	)
+	(via
 		(at 166.02744 82.714485)
 		(size 0.8)
@@
 	)
 	(via
+		(at 35.047115 81.386996)
+		(size 0.8)
+		(drill 0.4)
+		(layers "F.Cu" "B.Cu")
+		(free yes)
+		(net 3)
+	)
+	(via
 		(at 36.5125 30.1625)
 		(size 0.8)
@@
 	)
 	(segment
-		(start 265.092318 90.303579)
-		(end 265.092318 88.510421)
+		(start 186.56681 92.1289)
+		(end 186.56681 91.08059)
 		(width 0.2)
 		(layer "B.Cu")
@@
 	)
 	(segment
-		(start 187.7266 90.463045)
-		(end 187.7266 92.714974)
+		(start 187.311282 92.873372)
+		(end 186.56681 92.1289)
 		(width 0.2)
 		(layer "B.Cu")
@@
 	)
 	(segment
-		(start 265.092318 88.510421)
-		(end 256.38125 79.799353)
+		(start 187.7266 90.463045)
+		(end 187.7266 92.714974)
 		(width 0.2)
 		(layer "B.Cu")
@@
 	)
 	(segment
-		(start 187.568202 92.873372)
-		(end 187.311282 92.873372)
+		(start 187.7266 92.714974)
+		(end 187.568202 92.873372)
 		(width 0.2)
 		(layer "B.Cu")
@@
 	)
 	(segment
-		(start 195.639645 82.55)
-		(end 187.7266 90.463045)
+		(start 256.416424 79.799353)
+		(end 240.473215 79.799353)
 		(width 0.2)
 		(layer "B.Cu")
@@
 	)
 	(segment
-		(start 187.7266 92.714974)
-		(end 187.568202 92.873372)
+		(start 265.092318 90.303579)
+		(end 265.092318 88.475247)
 		(width 0.2)
 		(layer "B.Cu")
@@
 	)
 	(segment
-		(start 186.56681 92.1289)
-		(end 186.56681 91.08059)
+		(start 240.473215 79.799353)
+		(end 237.722567 82.55)
 		(width 0.2)
 		(layer "B.Cu")
@@
 	)
 	(segment
-		(start 240.473215 79.799353)
-		(end 237.722567 82.55)
+		(start 195.639645 82.55)
+		(end 187.7266 90.463045)
 		(width 0.2)
 		(layer "B.Cu")
@@
 	)
 	(segment
-		(start 256.38125 79.799353)
-		(end 240.473215 79.799353)
+		(start 187.568202 92.873372)
+		(end 187.311282 92.873372)
 		(width 0.2)
 		(layer "B.Cu")
@@
 	)
 	(segment
-		(start 187.311282 92.873372)
-		(end 186.56681 92.1289)
+		(start 265.092318 88.475247)
+		(end 256.416424 79.799353)
 		(width 0.2)
 		(layer "B.Cu")

Commit message: V1 completed
Routing:
- net Net-(U1-PB4): track 22.1 -> 27.8 mm
- net ROW3: track 388.7 -> 388.0 mm
- net COL12: track 196.5 -> 196.8 mm, vias 0 -> 1
- net GND: vias 421 -> 428
Other:
- board text added: "JLCJLCJLCJLC"
- board text added: "v1.1"
- board text removed: "og curves here!"
