File: Project/plate.kicad_pcb (KiCad board)
At the start: 2 copper layers, 257.2 x 76.2 mm, 121 parts, among them J1 JST SH, SW1 DFU, U1 STM32F072CBT6, U2 XC6206PxxxMR-Regulator_Linear, U3 74HC4051, U4 OPA354, U5 74HC4051

Commit message: plate work
Parts:
- added REF**: Value, cipulot_parts:ecs_plate_cut_1U, F.Cu at (27.0, 91.3)
- added REF**: Value, cipulot_parts:ecs_plate_cut_1U, F.Cu at (127.0, 53.2)
- added REF**: Value, cipulot_parts:ecs_plate_cut_1U, F.Cu at (198.4, 34.1)
- added REF**: Value, cipulot_parts:ecs_plate_cut_1U, F.Cu at (203.2, 53.2)
- added REF**: Value, cipulot_parts:ecs_plate_cut_1U, F.Cu at (165.1, 53.2)
- added REF**: Value, cipulot_parts:ecs_plate_cut_1U, F.Cu at (217.5, 34.1)
- added REF**: Value, cipulot_parts:ecs_plate_cut_1U, F.Cu at (117.5, 72.2)
- added REF**: Value, cipulot_parts:ecs_plate_cut_1U, F.Cu at (84.1, 34.1)
- added REF**: Value, cipulot_parts:ecs_plate_cut_1U, F.Cu at (34.1, 72.2)
- added REF**: Value, cipulot_parts:ecs_plate_cut_1U, F.Cu at (155.6, 72.2)
- added REF**: Value, cipulot_parts:ecs_plate_cut_1U, F.Cu at (60.3, 72.2)
- added REF**: Value, cipulot_parts:ecs_plate_cut_1U, F.Cu at (136.5, 72.2)
- added REF**: Value, cipulot_parts:ecs_plate_cut_1U, F.Cu at (50.8, 53.2)
- added REF**: Value, cipulot_parts:ecs_plate_cut_1U, F.Cu at (108.0, 53.2)
- added REF**: Value, cipulot_parts:ecs_plate_cut_1U, F.Cu at (65.1, 34.1)
- added REF**: Value, cipulot_parts:ecs_plate_cut_1U, F.Cu at (141.3, 34.1)
- added REF**: Value, cipulot_parts:ecs_plate_cut_1U, F.Cu at (29.4, 53.2)
- added REF**: Value, cipulot_parts:ecs_plate_cut_2U, F.Cu at (-109.5, 7.14)
- added REF**: Value, cipulot_parts:ecs_plate_cut_1U, F.Cu at (160.3, 34.1)
- added REF**: Value, cipulot_parts:ecs_plate_cut_1U, F.Cu at (79.4, 91.3)
- added REF**: Value, cipulot_parts:ecs_plate_cut_1U, F.Cu at (122.2, 34.1)
- added REF**: Value, cipulot_parts:ecs_pad_1U_no_ring, F.Cu at (46.0, 34.1)
- added REF**: Value, cipulot_parts:ecs_plate_cut_1U, F.Cu at (262.7, 53.2)
- added REF**: Value, cipulot_parts:ecs_pad_1U_no_ring, F.Cu at (69.8, 115.9)
- added REF**: Value, cipulot_parts:ecs_plate_cut_1U, F.Cu at (212.7, 72.2)
- added REF**: Value, cipulot_parts:ecs_pad_1U_no_ring, F.Cu at (65.1, 34.1)
- added REF**: Value, cipulot_parts:ecs_plate_cut_1U, F.Cu at (258.0, 72.2)
- added REF**: Value, cipulot_parts:ecs_plate_cut_1U, F.Cu at (69.8, 53.2)
- added REF**: Value, cipulot_parts:ecs_plate_cut_1U, F.Cu at (212.7, 91.3)
- added REF**: Value, cipulot_parts:ecs_plate_cut_1U, F.Cu at (231.8, 72.2)
- added REF**: Value, cipulot_parts:ecs_plate_cut_2U, F.Cu at (248.4, 72.2)
- added REF**: Value, cipulot_parts:ecs_plate_cut_1U, F.Cu at (174.6, 72.2)
- added REF**: Value, cipulot_parts:ecs_plate_cut_1U, F.Cu at (98.4, 72.2)
- added REF**: Value, cipulot_parts:ecs_plate_cut_1U, F.Cu at (146.1, 53.2)
- added REF**: Value, cipulot_parts:ecs_plate_cut_1U, F.Cu at (222.2, 53.2)
- added REF**: Value, cipulot_parts:ecs_plate_cut_1U, F.Cu at (236.5, 34.1)
- added REF**: Value, cipulot_parts:ecs_plate_cut_1U, F.Cu at (193.7, 72.2)
- added REF**: Value, cipulot_parts:ecs_plate_cut_1U, F.Cu at (103.2, 34.1)
- added REF**: Value, cipulot_parts:ecs_plate_cut_2U, F.Cu at (253.2, 53.2)
- added REF**: Value, cipulot_parts:ecs_plate_cut_1U, F.Cu at (174.6, 91.3)
- added REF**: Value, cipulot_parts:ecs_plate_cut_1U, F.Cu at (184.2, 53.2)
- added REF**: Value, cipulot_parts:ecs_plate_cut_1U, F.Cu at (179.4, 34.1)
- added REF**: Value, cipulot_parts:ecs_plate_cut_1U, F.Cu at (265.1, 91.3)
- added REF**: Value, cipulot_parts:ecs_plate_cut_2U, F.Cu at (262.7, 43.7)
- added REF**: Value, cipulot_parts:ecs_plate_cut_1U, F.Cu at (46.0, 34.1)
- added REF**: Value, cipulot_parts:ecs_plate_cut_1U, F.Cu at (241.3, 53.2)
- added REF**: Value, cipulot_parts:ecs_pad_1U_no_ring, F.Cu at (50.8, 115.9)
- added REF**: Value, cipulot_parts:ecs_plate_cut_1U, F.Cu at (60.3, 91.3)
- added REF**: Value, cipulot_parts:ecs_plate_cut_1U, F.Cu at (117.5, 91.3)
- added REF**: Value, cipulot_parts:ecs_plate_cut_1U, F.Cu at (27.0, 34.1)
- added REF**: Value, cipulot_parts:ecs_plate_cut_1U, F.Cu at (231.8, 91.3)
- added REF**: Value, cipulot_parts:ecs_plate_cut_1U, F.Cu at (79.4, 72.2)
- added REF**: Value, cipulot_parts:ecs_plate_cut_1U, F.Cu at (88.9, 53.2)
- added REF**: Value, cipulot_parts:ecs_plate_cut_1U, F.Cu at (260.4, 34.1)
- moved C1 0.23 mm to (92.5, 89.9)
- moved C7 0.23 mm to (92.5, 88.9)
Routing:
- net ROW0: track 428.4 -> 0.00 mm, vias 14 -> 0
- net ROW1: track 424.5 -> 0.00 mm, vias 20 -> 0
- net ROW3: track 397.8 -> 0.00 mm, vias 12 -> 0
- net ROW2: track 362.0 -> 0.00 mm, vias 16 -> 0
- net +3V3: track 275.4 -> 0.00 mm, vias 9 -> 0
- net APLEX_OUT: track 192.3 -> 0.00 mm, vias 5 -> 0
- net COL12: track 191.7 -> 0.00 mm, vias 5 -> 0
- net AMUX_SEL_0: track 172.7 -> 0.00 mm, vias 2 -> 0
- net AMUX_SEL_1: track 171.9 -> 0.00 mm, vias 2 -> 0
- net AMUX_SEL_2: track 171.1 -> 0.00 mm, vias 2 -> 0
- net COL11: track 161.8 -> 0.00 mm, vias 4 -> 0
- net COL5: track 141.4 -> 0.00 mm, vias 8 -> 0
- net COL4: track 137.0 -> 0.00 mm, vias 7 -> 0
- net D_P: track 121.3 -> 0.00 mm, vias 2 -> 0
- net D_N: track 117.6 -> 0.00 mm
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Other:
- board size 257.2 x 76.2 mm -> 634.4 x 233.1 mm
- board text added: "3U"
- board text added: "6U"
- board text added: "7U"
- board text added: "8U"
- board text added: "SCREW HOLES CHECK!!!!!! CUT OUT AND SWITCH POSITION CHECK!!! MULTIPLE OPTIONS BOTTOM ROW CHECK"
