File: Project/EC matrix.kicad_sch (KiCad schematic)
At the start: 50 parts

Commit message: pcb & plate revisions & firmware
Parts:
- SW_EC40, SW_EC49: footprint cipulot_parts:ecs_pad_no_ring_stepped&normal_cut -> cipulot_parts:ecs_pad_1U_no_ring
Changed lines of the file:
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@@
       (effects (font (size 1.27 1.27)) hide)
     )
-    (property "Footprint" "cipulot_parts:ecs_pad_no_ring_stepped&normal_cut" (at 215.265 86.995 0)
+    (property "Footprint" "cipulot_parts:ecs_pad_1U_no_ring" (at 215.265 86.995 0)
       (effects (font (size 1.27 1.27)) hide)
     )
@@
       (effects (font (size 1.27 1.27)) hide)
     )
-    (property "Footprint" "cipulot_parts:ecs_pad_no_ring_stepped&normal_cut" (at 55.245 86.995 0)
-      (effects (font (size 1.27 1.27)) hide)
-    )
+    (property "Footprint" "cipulot_parts:ecs_pad_1U_no_ring" (at 55.245 86.995 0)
+      (effects (font (size 1.27 1.27)) hide)
+    )
