File: Project/analog.kicad_sch (KiCad schematic)
At the start: 23 parts, among them U2 74HC4051, U4 74HC4051, U5 OPA354

Commit message: initialise
Parts:
- C11, C12, C9: value 100n -> 100nF
Changed lines of the file:
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@@
       (effects (font (size 1.27 1.27)))
     )
-    (property "Value" "100n" (at 193.802 27.7114 90)
+    (property "Value" "100nF" (at 193.802 27.7114 90)
       (effects (font (size 1.27 1.27)))
     )
@@
       (effects (font (size 1.27 1.27)))
     )
-    (property "Value" "100n" (at 95.25 18.7706 90)
+    (property "Value" "100nF" (at 95.25 18.7706 90)
       (effects (font (size 1.27 1.27)))
     )
@@
       (effects (font (size 1.27 1.27)))
     )
-    (property "Value" "100n" (at 95.25 83.5406 90)
-      (effects (font (size 1.27 1.27)))
-    )
+    (property "Value" "100nF" (at 95.25 83.5406 90)
+      (effects (font (size 1.27 1.27)))
+    )
