File: Project/Plates/6u ISO small mods.kicad_pcb (KiCad board)
At the start: 2 copper layers, 257.2 x 76.2 mm, 43 parts

Commit message: pcb & plate revisions & firmware
Parts:
- added REF**: Value, cipulot_parts:ecs_6U_space_stab, F.Cu at (146.1, 91.3)
- added REF**: Value, cipulot_parts:ecs_plate_cut_1U, F.Cu at (146.1, 91.3)
- added REF**: Value, cipulot_parts:ecs_plate_cut_6U_space_stab, F.Cu at (146.1, 91.3)
Other:
- outline, holes or cut-outs redrawn
- board text added: "REF**"
