File: Project/Plates/10u big mods.kicad_pcb (KiCad board)
At the start: 2 copper layers, 257.2 x 76.2 mm, 45 parts

Commit message: bottom row change, plate update, firmware update
Parts:
- removed the REF** at (146.1, 91.3) (x2)
- removed the REF** at (231.8, 91.3)
- removed the REF** at (79.4, 91.3)
- removed the REF** at (212.7, 91.3)
- removed the REF** at (241.3, 53.2)
- removed the REF** at (60.3, 91.3)
- added REF**: Value, cipulot_parts:ecs_plate_cut_7U_space_stab, F.Cu at (146.1, 91.3)
- added REF**: Value, cipulot_parts:ecs_7U_space_stab, F.Cu at (146.1, 91.3)
- added REF**: Value, cipulot_parts:ecs_plate_cut_1U, F.Cu at (260.4, 34.1)
- added SW_EC39: Topre, cipulot_parts:ecs_pad_1U_no_ring, F.Cu at (27.0, 91.3)
- moved REF** 13.5 mm to (253.2, 53.2), turned to 0 degrees
Other:
- outline, holes or cut-outs redrawn
- board text removed: "REF**"
